File: colorsound_wah/_autosave-colorsound_wah.kicad_pcb (KiCad board)
At the start: 2 copper layers, 36 parts, among them Q1 2N2222, SW1 SW_Wuerth_450301014042, U1 40106, U2 VTL5C9

Commit message: u
Parts:
- moved R3 104.2 mm to (200.6, 90.0), turned to 180 degrees
- moved R4 102.0 mm to (196.5, 103.6), turned to 90 degrees
- moved R2 100.1 mm to (197.5, 71.9), turned to -90 degrees
- moved R1 95.2 mm to (192.5, 71.9), turned to -90 degrees
- moved R6 91.4 mm to (187.5, 71.9), turned to -90 degrees
- moved C1 87.0 mm to (197.5, 69.5), turned to 180 degrees
- moved C8 86.2 mm to (196.0, 85.5), turned to 180 degrees
- moved R7 85.6 mm to (182.5, 82.1), turned to 90 degrees
- moved R8 83.0 mm to (177.0, 71.9), turned to -90 degrees
- moved C2 81.2 mm to (191.0, 95.5), turned to 180 degrees
- moved R9 81.0 mm to (177.1, 85.0), turned to 180 degrees
- moved R5 79.9 mm to (177.1, 89.0), turned to 180 degrees
- moved C4 76.7 mm to (187.5, 85.5), turned to 180 degrees
- moved C3 73.3 mm to (182.5, 69.5)
- moved C5 71.6 mm to (182.5, 90.0)
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Routing:
- net GND: track 0.00 -> 196.9 mm
- net VCC: track 0.00 -> 73.8 mm
- net Net-(D1-A): track 0.00 -> 64.0 mm
- net Net-(U2-+): track 0.00 -> 46.0 mm
- net Net-(Q1-B): track 0.00 -> 39.4 mm
- net Net-(C6-Pad1): track 0.00 -> 34.9 mm
- net Net-(C7-Pad2): track 0.00 -> 32.3 mm
- net Net-(SW1-A): track 0.00 -> 27.3 mm
- net Net-(R11-Pad1): track 0.00 -> 25.5 mm
- net Net-(Q1-C): track 0.00 -> 25.5 mm
- net Net-(SW1-B): track 0.00 -> 20.5 mm
- net Net-(C5-Pad2): track 0.00 -> 20.4 mm
- net Net-(SW1-C): track 0.00 -> 18.4 mm
- net Net-(C2-Pad2): track 0.00 -> 14.2 mm
- net Net-(R10-Pad1): track 0.00 -> 13.7 mm
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- added copper zone on B.Cu, net GND
Other:
- board outline added: 80 x 43 mm
