File: colorsound_wah/colorsound_wah.kicad_sch (KiCad schematic)
At the start: 25 parts, among them Q1 2N2222, SW1 SW_Wuerth_450301014042, U1 40106, U2 VTL5C

Commit message: UPDATE
Parts:
- added C7: 2.2n, Capacitor_THT:C_Rect_L7.0mm_W2.0mm_P5.00mm, symbol Device:C_Small
- added C8: 100n, Capacitor_THT:C_Rect_L7.0mm_W2.0mm_P5.00mm, symbol Device:C_Small
- added R12: 100K, Resistor_THT:R_Axial_DIN0207_L6.3mm_D2.5mm_P10.16mm_Horizontal, symbol Device:R_Small
- added RV4: 100K, Potentiometer_THT:Potentiometer_ACP_CA9-H5_Horizontal, symbol Device:R_Potentiometer_Small
- C1, C2: footprint (none) -> Capacitor_THT:C_Rect_L7.0mm_W2.0mm_P5.00mm
- C3: value 100n -> 15n; footprint (none) -> Capacitor_THT:C_Rect_L7.0mm_W2.0mm_P5.00mm
- C4, C5: value 100n -> 2.2n; footprint (none) -> Capacitor_THT:C_Rect_L7.0mm_W2.0mm_P5.00mm
- C6: value C_Polarized_Small -> 68u; footprint (none) -> Capacitor_THT:CP_Radial_D5.0mm_P2.00mm
- D1: footprint (none) -> LED_THT:LED_D2.0mm_W4.0mm_H2.8mm_FlatTop
- Q1: footprint Package_TO_SOT_THT:TO-39-3 -> Package_TO_SOT_THT:TO-92L_Inline_Wide
- R1, R2, R3, R4: footprint (none) -> Resistor_THT:R_Axial_DIN0207_L6.3mm_D2.5mm_P10.16mm_Horizontal
- R10: value 330K -> 2.2K; footprint (none) -> Resistor_THT:R_Axial_DIN0207_L6.3mm_D2.5mm_P10.16mm_Horizontal
- R11: value 330K -> 1K; footprint (none) -> Resistor_THT:R_Axial_DIN0207_L6.3mm_D2.5mm_P10.16mm_Horizontal
- R5: value 100K -> 47K; footprint (none) -> Resistor_THT:R_Axial_DIN0207_L6.3mm_D2.5mm_P10.16mm_Horizontal
- R6, R7: value 330K -> 180K; footprint (none) -> Resistor_THT:R_Axial_DIN0207_L6.3mm_D2.5mm_P10.16mm_Horizontal
- R8: value 330K -> 33K; footprint (none) -> Resistor_THT:R_Axial_DIN0207_L6.3mm_D2.5mm_P10.16mm_Horizontal
- R9: value 1M -> 33K; footprint (none) -> Resistor_THT:R_Axial_DIN0207_L6.3mm_D2.5mm_P10.16mm_Horizontal
- RV1: footprint (none) -> Potentiometer_THT:Potentiometer_ACP_CA9-H5_Horizontal
- RV2: value 100K -> 10K; footprint (none) -> Potentiometer_THT:Potentiometer_ACP_CA9-H5_Horizontal
- RV3: value 100K -> 25K; footprint (none) -> Potentiometer_THT:Potentiometer_ACP_CA9-H5_Horizontal
- U1: footprint (none) -> Package_DIP:CERDIP-14_W7.62mm_SideBrazed_LongPads_Socket
- U2: value VTL5C -> VTL5C9
Connections:
- net Output: now also RV4.2; no longer C2.2, R5.1
- net at C2.1, Q1.3 (C), R3.1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: now also C8.2; no longer C5.2, R7.1
- net GNDREF renamed GND
- net GND: now also RV4.3
- net VDD renamed VCC
- new net: C2.2, C7.1, R12.2
- new net: C5.2, C8.1, R7.1
- new net: C7.2, R12.1, R5.1, RV4.1
Other:
- moved on the sheet: C1, C2, C3, C4, C5, C6, D1, Q1, R1, R10, R11, R2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

Commit message: upodate
Parts:
- added H1: Input, TestPoint:TestPoint_Loop_D2.50mm_Drill1.0mm_LowProfile, symbol Mechanical:MountingHole_Pad
- added H2, H3, H4, H6: MountingHole_Pad, TestPoint:TestPoint_Loop_D2.50mm_Drill1.0mm_LowProfile, symbol Mechanical:MountingHole_Pad
- added H5: GND, TestPoint:TestPoint_Loop_D2.50mm_Drill1.0mm_LowProfile, symbol Mechanical:MountingHole_Pad
Connections:
- net GND: now also H4.1, H5.1, H6.1
- net Input guitar: now also H1.1
- net Output: now also H2.1
- net VCC: now also H3.1

Commit message: update
Parts:
- removed C6: 68u, Capacitor_THT:CP_Radial_D5.0mm_P2.00mm, symbol Device:C_Polarized_Small
- removed D1: LED, LED_THT:LED_D2.0mm_W4.0mm_H2.8mm_FlatTop, symbol Device:LED
- removed R10: 2.2K, Resistor_THT:R_Axial_DIN0207_L6.3mm_D2.5mm_P10.16mm_Horizontal, symbol Device:R_Small
- removed R11: 1K, Resistor_THT:R_Axial_DIN0207_L6.3mm_D2.5mm_P10.16mm_Horizontal, symbol Device:R_Small
- removed RV1: 100K, Potentiometer_THT:Potentiometer_ACP_CA9-H5_Horizontal, symbol Device:R_Potentiometer_Small
- removed RV2: 10K, Potentiometer_THT:Potentiometer_ACP_CA9-H5_Horizontal, symbol Device:R_Potentiometer_Small
- removed RV3: 25K, Potentiometer_THT:Potentiometer_ACP_CA9-H5_Horizontal, symbol Device:R_Potentiometer_Small
- removed SW1: SW_Wuerth_450301014042, Button_Switch_THT:SW_Slide-03_Wuerth-WS-SLTV_10x2.5x6.4_P2.54mm, symbol Switch:SW_Wuerth_450301014042
- removed U1: 40106, Package_DIP:CERDIP-14_W7.62mm_SideBrazed_LongPads_Socket, symbol 4xxx:40106
- removed U2: VTL5C9, OptoDevice:PerkinElmer_VTL5C, symbol Isolator:VTL5C
- added C10: 47u, LibraryGabi:CP_Radial_D5.0mm_P2.00mm, symbol Device:C_Polarized_Small
- added C9: 100n, Capacitor_THT:C_Disc_D11.0mm_W5.0mm_P5.00mm, symbol Device:C_Small
- added H7, H9: GND, LibraryGabi:TestPoint_Loop_D2.50mm_Drill1.85mm, symbol Mechanical:MountingHole_Pad
- added H8: POT, TestPoint:TestPoint_Loop_D2.50mm_Drill1.0mm_LowProfile, symbol Mechanical:MountingHole_Pad
- added R13: 1M, LibraryGabi:R_Axial_DIN0207_L6.3mm_D2.5mm_P10.16mm_Horizontal, symbol Device:R_Small
- C1, C2, C3, C4, C5, C7, C8: footprint Capacitor_THT:C_Rect_L7.0mm_W2.0mm_P5.00mm -> LibraryGabi:C_Rect_L7.0mm_W2.0mm_P5.00mm
- H2: value MountingHole_Pad -> Output
- H3: value MountingHole_Pad -> VCC
- H4, H6: value MountingHole_Pad -> GND; footprint TestPoint:TestPoint_Loop_D2.50mm_Drill1.0mm_LowProfile -> LibraryGabi:TestPoint_Loop_D2.50mm_Drill1.85mm
- H5: footprint TestPoint:TestPoint_Loop_D2.50mm_Drill1.0mm_LowProfile -> LibraryGabi:TestPoint_Loop_D2.50mm_Drill1.85mm
- R1, R12, R2, R4, R5, R6, R7, R8, R9: footprint Resistor_THT:R_Axial_DIN0207_L6.3mm_D2.5mm_P10.16mm_Horizontal -> LibraryGabi:R_Axial_DIN0207_L6.3mm_D2.5mm_P10.16mm_Horizontal
- R3: value 5.7M -> 2M; footprint Resistor_THT:R_Axial_DIN0207_L6.3mm_D2.5mm_P10.16mm_Horizontal -> LibraryGabi:R_Axial_DIN0207_L6.3mm_D2.5mm_P10.16mm_Horizontal
- RV4: footprint Potentiometer_THT:Potentiometer_ACP_CA9-H5_Horizontal -> LibraryGabi:Potentiometer_ACP_CA9-H5_Horizontal
Connections:
- net GND: now also C10.2, C9.1, H7.1, H9.1
- net VCC: now also C10.1, C9.2
- net at R9.2: now also H8.1
- net at C4.1, Q1.2 (B), R1.1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: now also R13.2; no longer R3.2
- new net: R13.1, R3.2
Other:
- moved on the sheet: C1, C2, C3, C4, C5, C7, C8, H1, H2, H3, H4, H5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
